Commit message: locomotion achieved

File: resources/robots/m2/urdf/SVANM2_URDF.urdf (robot description, URDF)
Before this commit: robot svan_urdf_package, 18 links, 17 joints
Links:
- link FL_calf: mass 0.2002422228142348 -> 0.2; geometry collision mesh filename=../meshes/LF_SHANK.STL; visual mesh filename=../meshes/LF_SHANK.STL
- link FL_hip: mass 1.349989526327068 -> 1.35; geometry collision mesh filename=../meshes/LF_HIP.STL; visual mesh filename=../meshes/LF_HIP.STL
- link FL_thigh: mass 0.25008571121327 -> 0.25; geometry collision mesh filename=../meshes/LF_THIGH.STL; visual mesh filename=../meshes/LF_THIGH.STL
- link FR_calf: mass 0.2002422228142348 -> 0.2; geometry collision mesh filename=../meshes/RF_SHANK.STL; visual mesh filename=../meshes/RF_SHANK.STL
- link FR_hip: mass 1.3499526327116 -> 1.35; geometry collision mesh filename=../meshes/RF_HIP.STL; visual mesh filename=../meshes/RF_HIP.STL
- link FR_thigh: mass 0.25008571121328 -> 0.25; geometry collision mesh filename=../meshes/RF_THIGH.STL; visual mesh filename=../meshes/RF_THIGH.STL
- link RL_calf: mass 0.2002422228142348 -> 0.2; geometry collision mesh filename=../meshes/LH_SHANK.STL; visual mesh filename=../meshes/LH_SHANK.STL
- link RL_hip: mass 1.349959526327067 -> 1.35; geometry collision mesh filename=../meshes/LH_HIP.STL; visual mesh filename=../meshes/LH_HIP.STL
- link RL_thigh: mass 0.25008560926126 -> 0.25; geometry collision mesh filename=../meshes/LH_THIGH.STL; visual mesh filename=../meshes/LH_THIGH.STL
- link RR_calf: mass 0.2002422228142348 -> 0.2; geometry collision mesh filename=../meshes/RH_SHANK.STL; visual mesh filename=../meshes/RH_SHANK.STL
- link RR_hip: mass 1.349959526327114 -> 1.35; geometry collision mesh filename=../meshes/RH_HIP.STL; visual mesh filename=../meshes/RH_HIP.STL
- link RR_thigh: mass 0.25008571121328 -> 0.25; geometry collision mesh filename=../meshes/RH_THIGH.STL; visual mesh filename=../meshes/RH_THIGH.STL
- link trunk: mass 3.423410872609609 -> 3.4234; geometry collision mesh filename=../meshes/BASE.STL; visual mesh filename=../meshes/BASE.STL
Joints:
- joint FL_calf_joint: origin xyz=0.0041389 -0.01 -0.16494 rpy=0 0 0 -> xyz=0 0 -0.1915 rpy=0 0 0
- joint FL_hip_joint: origin xyz=0.20368 0.06 0 rpy=0 0 0 -> xyz=0.155 0.06 0 rpy=0 0 0
- joint FL_thigh_joint: origin xyz=0.043 0.07525 0 rpy=0 0 0 -> xyz=0.043751 0.0796 0 rpy=0 0 0
- joint FR_calf_joint: origin xyz=0.0041389 0.01 -0.16494 rpy=0 0 0 -> xyz=0 0 -0.1915 rpy=0 0 0
- joint FR_hip_joint: origin xyz=0.20368 -0.06 0 rpy=0 0 0 -> xyz=0.155 -0.06 0 rpy=0 0 0
- joint FR_thigh_joint: origin xyz=0.043 -0.07525 0 rpy=0 0 0 -> xyz=0.043751 -0.0796 0 rpy=0 0 0
- joint RL_calf_joint: origin xyz=-0.0038618 -0.01 -0.16493 rpy=0 0 0 -> xyz=0 0 -0.1915 rpy=0 0 0
- joint RL_hip_joint: origin xyz=-0.20482 0.06 0 rpy=0 0 0 -> xyz=-0.155 0.06 0 rpy=0 0 0
- joint RL_thigh_joint: origin xyz=-0.043 0.07525 0 rpy=0 0 0 -> xyz=-0.043751 0.0796 0 rpy=0 0 0
- joint RR_calf_joint: origin xyz=-0.0038618 0.01 -0.16493 rpy=0 0 0 -> xyz=0 0 -0.1915 rpy=0 0 0
- joint RR_hip_joint: origin xyz=-0.20482 -0.06 0 rpy=0 0 0 -> xyz=-0.155 -0.06 0 rpy=0 0 0
- joint RR_thigh_joint: origin xyz=-0.043 -0.07525 0 rpy=0 0 0 -> xyz=-0.043751 -0.0796 0 rpy=0 0 0

File: resources/robots/svan_m2/urdf/svan_urdf_package copy.urdf (robot description, URDF)
Before this commit: robot svan_urdf_package, 18 links, 17 joints
Links:
- link FL_calf: mass 0.2002422228142348 -> 0.122422228142348
- link FL_hip: mass 1.349989526327068 -> 0.547089526327068
- link FL_thigh: mass 0.25008571121327 -> 0.147108571121327
- link FR_calf: mass 0.2002422228142348 -> 0.122422228142348
- link FR_hip: mass 1.3499526327116 -> 0.547089526327116
- link FR_thigh: mass 0.25008571121328 -> 0.147108571121328
- link RL_calf: mass 0.2002422228142348 -> 0.122422317176859
- link RL_hip: mass 1.349959526327067 -> 0.547089526327067
- link RL_thigh: mass 0.25008560926126 -> 0.147108560926126
- link RR_calf: mass 0.2002422228142348 -> 0.122422246876929
- link RR_hip: mass 1.349959526327114 -> 0.547089526327114
- link RR_thigh: mass 0.25008571121328 -> 0.147108571121328
- link trunk: mass 3.423410872609609 -> 2.99710872609609

Commit message: perturbations added

File: resources/robots/m2/urdf/SVANM2_URDF.urdf (robot description, URDF)
Before this commit: robot SVANM2_URDF, 18 links, 17 joints
Links:
- link FL_calf: mass 0.2 -> 0.2017400
- link FL_hip: mass 1.35 -> 1.3509490
- link FL_thigh: mass 0.25 -> 0.2502465
- link FR_calf: mass 0.2 -> 0.2017400
- link FR_hip: mass 1.35 -> 1.3509490
- link FR_thigh: mass 0.25 -> 0.2502465
- link RL_calf: mass 0.2 -> 0.2017400
- link RL_hip: mass 1.35 -> 1.3509490
- link RL_thigh: mass 0.25 -> 0.2502465
- link RR_calf: mass 0.2 -> 0.2017400
- link RR_hip: mass 1.35 -> 1.3509490
- link RR_thigh: mass 0.25 -> 0.2502465

Commit message: updated urdf, training not happening

File: resources/robots/m2/urdf/SVANM2_URDF.urdf (robot description, URDF)
Before this commit: robot SVANM2_URDF, 18 links, 17 joints
Links:
- link FL_foot: geometry collision sphere radius=0.02; visual sphere radius=0.02
- link FR_foot: geometry collision sphere radius=0.02; visual sphere radius=0.02
- link RL_foot: geometry collision sphere radius=0.02; visual sphere radius=0.02
- link RR_foot: geometry collision sphere radius=0.02; visual sphere radius=0.02
- link trunk: mass 3.4234 -> 3.4234000
Joints:
- joint FL_foot_fixed: origin xyz=-0.026618 0 -0.16693 rpy=0 0 0 -> xyz=-0.0 0 -0.16693 rpy=0 0 0
- joint FR_foot_fixed: origin xyz=-0.026457 0 -0.16693 rpy=0 0 0 -> xyz=-0.0 0 -0.16693 rpy=0 0 0
- joint RL_foot_fixed: origin xyz=-0.0185 0 -0.16802 rpy=0 0 0 -> xyz=-0.0 0 -0.16802 rpy=0 0 0
- joint RR_foot_fixed: origin xyz=-0.018339 0 -0.16802 rpy=0 0 0 -> xyz=-0.0 0 -0.16802 rpy=0 0 0

Commit message: training with terrains + level conditions + rigid shape dynamics levels + mass randomization at initialization

File: resources/robots/m2/urdf/SVANM2_URDF.urdf (robot description, URDF)
Before this commit: robot SVANM2_URDF, 18 links, 17 joints
Links:
- link FL_foot: geometry collision sphere radius=0.01; visual sphere radius=0.01
- link FR_foot: geometry collision sphere radius=0.01; visual sphere radius=0.01
- link RL_foot: geometry collision sphere radius=0.01; visual sphere radius=0.01
- link RR_foot: geometry collision sphere radius=0.01; visual sphere radius=0.01
- link trunk: mass 3.4234000 -> 3.4234
Joints:
- joint FL_foot_fixed: origin xyz=-0.0 0 -0.16693 rpy=0 0 0 -> xyz=-0.026618 0 -0.16693 rpy=0 0 0
- joint FR_foot_fixed: origin xyz=-0.0 0 -0.16693 rpy=0 0 0 -> xyz=-0.026457 0 -0.16693 rpy=0 0 0
- joint RL_foot_fixed: origin xyz=-0.0 0 -0.16802 rpy=0 0 0 -> xyz=-0.0185 0 -0.16802 rpy=0 0 0
- joint RR_foot_fixed: origin xyz=-0.0 0 -0.16802 rpy=0 0 0 -> xyz=-0.018339 0 -0.16802 rpy=0 0 0
