Commit message: urdf limits expanded, inertias fixed. Training happening

File: resources/robots/m2/urdf/SVANM2_URDF_apt.urdf (robot description, URDF)
Before this commit: robot SVANM2_URDF, 18 links, 17 joints
Links:
- link FL_foot: geometry collision sphere radius=0.02; visual sphere radius=0.02
- link FR_foot: geometry collision sphere radius=0.02; visual sphere radius=0.02
- link RL_foot: geometry collision sphere radius=0.02; visual sphere radius=0.02
- link RR_foot: geometry collision sphere radius=0.02; visual sphere radius=0.02
Joints:
- joint FL_foot_fixed: origin xyz=-0.026618 0 -0.16693 rpy=0 0 0 -> xyz=-0.0 0 -0.16693 rpy=0 0 0
- joint FR_foot_fixed: origin xyz=-0.026457 0 -0.16693 rpy=0 0 0 -> xyz=-0.0 0 -0.16693 rpy=0 0 0
- joint RL_foot_fixed: origin xyz=-0.0185 0 -0.16802 rpy=0 0 0 -> xyz=-0.0 0 -0.16802 rpy=0 0 0
- joint RR_foot_fixed: origin xyz=-0.018339 0 -0.16802 rpy=0 0 0 -> xyz=-0.0 0 -0.16802 rpy=0 0 0

File: resources/robots/m2/urdf/SVANM2_URDF_apt_prev.urdf (robot description, URDF)
Before this commit: robot SVANM2_URDF, 18 links, 17 joints
Joints:
- joint FL_foot_fixed: origin xyz=-0.026618 0 -0.16693 rpy=0 0 0 -> xyz=-0.0 0 -0.16693 rpy=0 0 0
- joint FR_foot_fixed: origin xyz=-0.026457 0 -0.16693 rpy=0 0 0 -> xyz=-0.0 0 -0.16693 rpy=0 0 0
- joint RL_foot_fixed: origin xyz=-0.0185 0 -0.16802 rpy=0 0 0 -> xyz=-0.0 0 -0.16802 rpy=0 0 0
- joint RR_foot_fixed: origin xyz=-0.018339 0 -0.16802 rpy=0 0 0 -> xyz=-0.0 0 -0.16802 rpy=0 0 0

File: resources/robots/m2/urdf/SVANM2_URDF_inertia_change.urdf (robot description, URDF)
Before this commit: robot SVANM2_URDF, 18 links, 17 joints
Links:
- link FL_foot: geometry collision sphere radius=0.02; visual sphere radius=0.02
- link FR_foot: geometry collision sphere radius=0.02; visual sphere radius=0.02
- link RL_foot: geometry collision sphere radius=0.02; visual sphere radius=0.02
- link RR_foot: geometry collision sphere radius=0.02; visual sphere radius=0.02
Joints:
- joint FL_calf_joint: limit lower=-2.69653369433 upper=-0.916297857297 effort=55 velocity=28.6 -> lower=-4.69653369433 upper=4.916297857297 effort=55 velocity=28.6
- joint FL_hip_joint: limit lower=-0.802851455917 upper=0.802851455917 effort=20 velocity=52.4 -> lower=-3.802851455917 upper=3.802851455917 effort=20 velocity=52.4
- joint FL_thigh_joint: limit lower=-1.0471975512 upper=4.18879020479 effort=55 velocity=28.6 -> lower=-4.0471975512 upper=4.18879020479 effort=55 velocity=28.6
- joint FR_calf_joint: limit lower=-2.69653369433 upper=-0.916297857297 effort=55 velocity=28.6 -> lower=-4.69653369433 upper=4.916297857297 effort=55 velocity=28.6
- joint FR_hip_joint: limit lower=-0.8 upper=0.8 effort=20 velocity=52.4 -> lower=-4.8 upper=4.8 effort=20 velocity=52.4
- joint FR_thigh_joint: limit lower=-1.0471975512 upper=4.18879020479 effort=55 velocity=28.6 -> lower=-4.0471975512 upper=4.18879020479 effort=55 velocity=28.6
- joint RL_calf_joint: limit lower=-2.69653369433 upper=-0.916297857297 effort=55 velocity=28.6 -> lower=-4.69653369433 upper=4.916297857297 effort=55 velocity=28.6
- joint RL_hip_joint: limit lower=-0.802851455917 upper=0.802851455917 effort=20 velocity=52.4 -> lower=-4.802851455917 upper=4.802851455917 effort=20 velocity=52.4
- joint RL_thigh_joint: limit lower=-1.0471975512 upper=4.18879020479 effort=55 velocity=28.6 -> lower=-4.0471975512 upper=4.18879020479 effort=55 velocity=28.6
- joint RR_calf_joint: limit lower=-2.69653369433 upper=-0.916297857297 effort=55 velocity=28.6 -> lower=-4.69653369433 upper=4.916297857297 effort=55 velocity=28.6
- joint RR_hip_joint: limit lower=-0.802851455917 upper=0.802851455917 effort=20 velocity=52.4 -> lower=-4.802851455917 upper=4.802851455917 effort=20 velocity=52.4
- joint RR_thigh_joint: limit lower=-1.0471975512 upper=4.18879020479 effort=55 velocity=28.6 -> lower=-4.0471975512 upper=4.18879020479 effort=55 velocity=28.6
