Commit message: Simulation trains with cpu

File: resources/robots/m2/urdf/SVANM2_URDF_inertia_change.urdf (robot description, URDF)
Before this commit: robot SVANM2_URDF, 18 links, 17 joints
Joints:
- removed joint FR_foot_fixed
- added joint fr_dummy_j: type fixed, parent FR_calf, child FR_foot, origin xyz=-0.0 0 -0.16693 rpy=0 0 0
- joint FL_foot_fixed: origin xyz=-0.026618 0 -0.16693 rpy=0 0 0 -> xyz=-0.0 0 -0.16693 rpy=0 0 0
- joint RL_foot_fixed: origin xyz=-0.0185 0 -0.16802 rpy=0 0 0 -> xyz=-0.0 0 -0.16802 rpy=0 0 0
- joint RR_foot_fixed: origin xyz=-0.018339 0 -0.16802 rpy=0 0 0 -> xyz=-0.0 0 -0.16802 rpy=0 0 0

Commit message: fixed the foot problem completely. made it little larger to ensure contact happens with foot and not the shank

File: resources/robots/m2/urdf/SVANM2_URDF_inertia_change.urdf (robot description, URDF)
Before this commit: robot SVANM2_URDF, 18 links, 17 joints
Links:
- link FL_foot: geometry collision sphere radius=0.022; visual sphere radius=0.022
- link FR_foot: geometry collision sphere radius=0.022; visual sphere radius=0.022
- link RL_foot: geometry collision sphere radius=0.022; visual sphere radius=0.022
- link RR_foot: geometry collision sphere radius=0.022; visual sphere radius=0.022
Joints:
- joint FL_calf_joint: limit lower=-4.69653369433 upper=4.916297857297 effort=55 velocity=28.6 -> lower=-4.69653369433 upper=4.916297857297 effort=55 velocity=10.6
- joint FL_hip_joint: limit lower=-3.802851455917 upper=3.802851455917 effort=20 velocity=52.4 -> lower=-3.802851455917 upper=3.802851455917 effort=20 velocity=10.4
- joint FL_thigh_joint: limit lower=-4.0471975512 upper=4.18879020479 effort=55 velocity=28.6 -> lower=-4.0471975512 upper=4.18879020479 effort=55 velocity=10.6
- joint FR_calf_joint: limit lower=-4.69653369433 upper=4.916297857297 effort=55 velocity=28.6 -> lower=-4.69653369433 upper=4.916297857297 effort=55 velocity=10.6
- joint FR_hip_joint: limit lower=-4.8 upper=4.8 effort=20 velocity=52.4 -> lower=-4.8 upper=4.8 effort=20 velocity=10.4
- joint FR_thigh_joint: limit lower=-4.0471975512 upper=4.18879020479 effort=55 velocity=28.6 -> lower=-4.0471975512 upper=4.18879020479 effort=55 velocity=10.6
- joint RL_calf_joint: limit lower=-4.69653369433 upper=4.916297857297 effort=55 velocity=28.6 -> lower=-4.69653369433 upper=4.916297857297 effort=55 velocity=10.6
- joint RL_hip_joint: limit lower=-4.802851455917 upper=4.802851455917 effort=20 velocity=52.4 -> lower=-4.802851455917 upper=4.802851455917 effort=20 velocity=10.4
- joint RL_thigh_joint: limit lower=-4.0471975512 upper=4.18879020479 effort=55 velocity=28.6 -> lower=-4.0471975512 upper=4.18879020479 effort=55 velocity=10.6
- joint RR_calf_joint: limit lower=-4.69653369433 upper=4.916297857297 effort=55 velocity=28.6 -> lower=-4.69653369433 upper=4.916297857297 effort=55 velocity=10.6
- joint RR_hip_joint: limit lower=-4.802851455917 upper=4.802851455917 effort=20 velocity=52.4 -> lower=-4.802851455917 upper=4.802851455917 effort=20 velocity=10.4
- joint RR_thigh_joint: limit lower=-4.0471975512 upper=4.18879020479 effort=55 velocity=28.6 -> lower=-4.0471975512 upper=4.18879020479 effort=55 velocity=10.6

Commit message: mcp running on svan in this quadruped

File: resources/robots/m2/urdf/SVANM2_URDF_inertia_change.urdf (robot description, URDF)
Before this commit: robot SVANM2_URDF, 18 links, 17 joints
Links:
- link FL_foot: mass 0.025 -> 0.06; geometry collision sphere radius=0.03; visual sphere radius=0.022
- link FR_foot: mass 0.025 -> 0.06; geometry collision sphere radius=0.03; visual sphere radius=0.022
- link RL_foot: mass 0.025 -> 0.06; geometry collision sphere radius=0.03; visual sphere radius=0.022
- link RR_foot: mass 0.025 -> 0.06; geometry collision sphere radius=0.03; visual sphere radius=0.022

Commit message: latest changes before merger with wtw dynamic randomizations and terrains

File: resources/robots/m2/urdf/SVANM2_URDF_inertia_change.urdf (robot description, URDF)
Before this commit: robot SVANM2_URDF, 18 links, 17 joints
Joints:
- joint FL_hip_joint: limit lower=-3.802851455917 upper=3.802851455917 effort=20 velocity=10.4 -> lower=-0.7 upper=0.7 effort=20 velocity=10.4
- joint FR_hip_joint: limit lower=-4.8 upper=4.8 effort=20 velocity=10.4 -> lower=-0.7 upper=0.7 effort=20 velocity=10.4
- joint RL_hip_joint: limit lower=-4.802851455917 upper=4.802851455917 effort=20 velocity=10.4 -> lower=-0.7 upper=0.7 effort=20 velocity=10.4
- joint RR_hip_joint: limit lower=-4.802851455917 upper=4.802851455917 effort=20 velocity=10.4 -> lower=-0.7 upper=0.7 effort=20 velocity=10.4

Commit message: training accomplished fairly well for non-base vel, important changes in play.py to fix unexplained signed changes. m2_flat config now includes some dof limit properties and rewards to acheive the same. urdf has some changed dof limits to provide limits to legged gym. observation space changed in legged robot compute obs.

File: resources/robots/m2/urdf/SVANM2_URDF_inertia_change.urdf (robot description, URDF)
Before this commit: robot SVANM2_URDF, 18 links, 17 joints
Joints:
- joint FL_calf_joint: limit lower=-4.69653369433 upper=4.916297857297 effort=55 velocity=10.6 -> lower=-4.69653369433 upper=4.916297857297 effort=35 velocity=10.6
- joint FL_thigh_joint: limit lower=-4.0471975512 upper=4.18879020479 effort=55 velocity=10.6 -> lower=-4.0471975512 upper=4.18879020479 effort=35 velocity=10.6
- joint FR_calf_joint: limit lower=-4.69653369433 upper=4.916297857297 effort=55 velocity=10.6 -> lower=-4.69653369433 upper=4.916297857297 effort=35 velocity=10.6
- joint FR_thigh_joint: limit lower=-4.0471975512 upper=4.18879020479 effort=55 velocity=10.6 -> lower=-4.0471975512 upper=4.18879020479 effort=35 velocity=10.6
- joint RL_calf_joint: limit lower=-4.69653369433 upper=4.916297857297 effort=55 velocity=10.6 -> lower=-4.69653369433 upper=4.916297857297 effort=35 velocity=10.6
- joint RL_thigh_joint: limit lower=-4.0471975512 upper=4.18879020479 effort=55 velocity=10.6 -> lower=-4.0471975512 upper=4.18879020479 effort=35 velocity=10.6
- joint RR_calf_joint: limit lower=-4.69653369433 upper=4.916297857297 effort=55 velocity=10.6 -> lower=-4.69653369433 upper=4.916297857297 effort=35 velocity=10.6
- joint RR_thigh_joint: limit lower=-4.0471975512 upper=4.18879020479 effort=55 velocity=10.6 -> lower=-4.0471975512 upper=4.18879020479 effort=35 velocity=10.6
